File: jake-projects.kicad_sch (KiCad schematic)
At the start: 12 parts, among them J1 Conn_01x02_Pin, SW1 ;-;, SW2 SW_Push, SW4 SW_SPST, U2 ATtiny85-20P

Commit message: revised/final draft of schematic + pcb
Parts:
- D1, SW1: value ;-; -> usr
Other:
- note removed: "Error: U1 pad 21 not found in Package_DIP:DIP-8_W7.62mm_Socket. Error: U1 pad 11 not found in Package_DIP:DIP-8_W7.62mm_Socket. Error: U1 pad 15 not found in Package_DIP:DIP-8_W7.62mm_Socket. Error: U1 pad 9 not found in Package_DIP:DIP-8_W7.62mm_Socket. Error: U1 pad 10 not found in Package_DIP:DIP-8_W7.62mm_Socket. Error: U1 pad 13 not found in Package_DIP:DIP-8_W7.62mm_Socket. Error: U1 pad 16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"
- note removed: "i forget why we decided to use this switch instead of the SPST (the one that didnt have two outputs)"
- note removed: "sorry jake i kinda took "inspiration" here from yours (in regards to the reset stuff) update: also the decoupling capacitor :/"
Changed lines of the file:
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@@
 		(company "lake electrical club")
-	)
-	(text "i forget why we decided to \nuse this switch instead of \nthe SPST (the one that didnt \nhave two outputs)"
-		(exclude_from_sim no)
-		(at 123.698 105.664 0)
-		(effects
-			(font
-				(size 1.27 1.27)
-			)
-		)
-	)
-	(text "sorry jake i kinda took \"inspiration\" here from yours (in regards to the reset stuff)\nupdate: also the decoupling capacitor :/"
-		(exclude_from_sim no)
-		(at 189.23 94.996 0)
-		(effects
-			(font
-				(size 1.27 1.27)
-			)
-		)
-	)
-	(text "Error: U1 pad 21 not found in Package_DIP:DIP-8_W7.62mm_Socket.\nError: U1 pad 11 not found in Package_DIP:DIP-8_W7.62mm_Socket.\nError: U1 pad 15 not found in Package_DIP:DIP-8_W7.62mm_Socket.\nError: U1 pad 9 not found in Package_DIP:DIP-8_W7.62mm_Socket.\nError: U1 pad 10 not found in Package_DIP:DIP-8_W7.62mm_Socket.\nError: U1 pad 13 not found in Package_DIP:DIP-8_W7.62mm_Socket.\nError: U1 pad 16 not found in Package_DIP:DIP-8_W7.62mm_Socket.\nError: U1 pad 17 not found in Package_DIP:DIP-8_W7.62mm_Socket.\nError: U1 pad 18 not found in Package_DIP:DIP-8_W7.62mm_Socket.\nError: U1 pad 19 not found in Package_DIP:DIP-8_W7.62mm_Socket.\nError: U1 pad 20 not found in Package_DIP:DIP-8_W7.62mm_Socket.\nError: U1 pad 14 not found in Package_DIP:DIP-8_W7.62mm_Socket.\nError: U1 pad 12 not found in Package_DIP:DIP-8_W7.62mm_Socket."
-		(exclude_from_sim no)
-		(at 72.898 46.482 0)
-		(effects
-			(font
-				(size 1.27 1.27)
-			)
-		)
 	)
 	(junction
@@
 			)
 		)
-		(property "Value" ";-;"
+		(property "Value" "usr"
 			(at 228.854 117.856 0)
 			(effects
@@
 			)
 		)
-		(property "Value" ";-;"
+		(property "Value" "usr"
 			(at 229.87 135.89 0)
 			(effects
